Commit message: working urdf and ikpy

File: spot-arm/Assets/StreamingAssets/ikpy/robot2.urdf (robot description, URDF)
Before this commit: robot spot_arm, 8 links, 7 joints
Joints:
- removed joint Rev10
- removed joint Rev11
- removed joint Rev3
- removed joint Rev6
- removed joint Rev7
- removed joint Rev8
- removed joint Rev9
- added joint j0: type revolute, parent base_link, child Part0_1, origin xyz=0.0 0.0 0.065 rpy=0 0 0, axis 0.0 0.0 1.0, limit lower=-3.141593 upper=2.617994 effort=100 velocity=100
- added joint j1: type revolute, parent Part0_1, child Part1_1, origin xyz=0.015 0.0 0.05 rpy=3.1415 0 0, axis -1.0 0.0 0.0, limit lower=-0.523598 upper=3.1415926 effort=100 velocity=100
- added joint j2: type revolute, parent Part1_1, child Part2_1, origin xyz=0.002 0.3125 0.0 rpy=0 0 0, axis 1.0 0.0 0.0, limit lower=0.0 upper=2.96706 effort=100 velocity=100
- added joint j3: type revolute, parent Part2_1, child Part3_1, origin xyz=-0.018 0.138 -0.0675 rpy=0 0 0, axis 0.0 1.0 0.0, limit lower=-2.879793 upper=2.879793 effort=100 velocity=100
- added joint j4: type revolute, parent Part3_1, child Part4_1, origin xyz=-0.0475 0.24809 0.0 rpy=0 0 0, axis 1.0 0.0 0.0, limit lower=-1.8326 upper=1.8326 effort=100 velocity=100
- added joint j5: type revolute, parent Part4_1, child gripper_1, origin xyz=0.04 0.081 0.0 rpy=0 0 0, axis -0.0 1.0 0.0, limit lower=-2.96706 upper=2.96706 effort=100 velocity=100
- added joint j6: type revolute, parent gripper_1, child finger_1, origin xyz=0 0.043915 -0.029 rpy=0 0 0, axis 1.0 -0.0 0.0, limit lower=-1.396263 upper=0.349066 effort=100 velocity=100
