Commit message: updated assets

File: spot-arm/Assets/StreamingAssets/ikpy/arm.urdf (robot description, URDF)
Before this commit: robot spot, 9 links, 8 joints
Links:
- removed link arm0.link_el0
- removed link arm0.link_el1
- removed link arm0.link_fngr
- removed link arm0.link_hr0
- removed link arm0.link_sh0
- removed link arm0.link_sh1
- removed link arm0.link_wr0
- removed link arm0.link_wr1
- added link finger
- added link gripper; visual mesh filename=link_models/arm0.link_wr1.obj.dae
- added link link1
- added link link2
- added link link3
- added link link4
- added link link5
- added link link6
- link base_link: geometry 
Joints:
- removed joint arm0.el0
- removed joint arm0.el1
- removed joint arm0.hr0
- removed joint arm0.sh0
- removed joint arm0.sh1
- removed joint arm0.wr0
- removed joint arm0.wr1
- added joint joint1: type revolute, parent base_link, child link1, origin xyz=0.292 0.0 0.188 rpy=0 0 0, axis 0 0 1, limit lower=-2.61799387799149441136 upper=3.14159265358979311599 effort=1000 velocity=1000.00
- added joint joint2: type revolute, parent link1, child link2, origin xyz=0.0 0.0 0.0 rpy=0 0 0, axis 0 1 0, limit lower=-3.14159265358979311599 upper=0.52359877559829881565 effort=1000 velocity=1000.00
- added joint joint2a: type revolute, parent link2, child link3, origin xyz=0.0 0.0 0.0 rpy=0 0 0, axis 1 0 0
- added joint joint3: type revolute, parent link3, child link4, origin xyz=0.3385 0 0 rpy=0 0 0, axis 0 1 0, limit lower=0 upper=3.14159265358979311599 effort=1000 velocity=1000.00
- added joint joint4: type revolute, parent link4, child link5, origin xyz=0.40330 0.0 0.0750 rpy=0 0 0, axis 1 0 0, limit lower=-2.79252680319092716487 upper=2.79252680319092716487 effort=1000 velocity=1000.00
- added joint joint5: type revolute, parent link5, child link6, origin xyz=0.0 0.0 0.0 rpy=0 0 0, axis 0 1 0, limit lower=-1.83259571459404613236 upper=1.83259571459404613236 effort=1000 velocity=1000.00
- added joint joint6: type revolute, parent link6, child gripper, origin xyz=0.0 0.0 0.0 rpy=0 0 0, axis 1 0 0, limit lower=-2.87979326579064354163 upper=2.87979326579064354163 effort=1000 velocity=1000.00
- joint arm0.f1x: child arm0.link_fngr -> finger; parent arm0.link_wr1 -> gripper

File: spot-arm/Assets/StreamingAssets/ikpy/robot2.urdf (robot description, URDF)
Before this commit: robot spot_arm, 8 links, 7 joints
Links:
- link Part0_1: mass 6.925827706354272 -> None; geometry 
- link Part1_1: mass 12.658281999999998 -> None; geometry 
- link Part2_1: mass 7.368455487741179 -> None; geometry 
- link Part3_1: mass 10.95245995004642 -> None; geometry 
- link Part4_1: mass 3.2278801394086396 -> None; geometry 
- link base_link: mass 5.770791545379091 -> None; geometry 
- link finger_1: mass 1.71236178687828 -> None; geometry 
- link gripper_1: mass 5.9780007036604434 -> None; geometry 
